File: voyager60NOCAPSLOCKLED.kicad_pcb (KiCad board)
At the start: 2 copper layers, 285 x 95.1 mm, 265 parts, among them Q1 2N7002, SW1 5.2x5.2mm, U1 ATmega32U4-MU, U2 PRTR5V0U2X, Y1 16Mhz

Commit message: Alps Stepped Caps Lock
Added alps stepped caps lock support at the cost of removing caps lock LED support.
Parts:
- removed G***: LOGO, locallib:ai-ring-6mm
- removed G***: LOGO, locallib:ai-ring-6mm-FancyAss
- removed G***: LOGO, locallib:ai-ring-6mm-FancyAss-Mask
- removed the REF** at (36.5, 69.8)
- added K_CAPS3: MX-1.5U, MX_Alps_Hybrid:ALPS-1.5U, F.Cu at (36.5, 69.8)
Routing:
- net +5V: track 1811.3 -> 1759.6 mm, vias 14 -> 13
- net Net-(D31-Pad2): track 17.5 -> 27.6 mm
- net COL0: track 118.7 -> 124.1 mm
- net LEDGND: track 1407.5 -> 1405.2 mm
