File: Voyager60.kicad_pcb (KiCad board)
At the start: 2 copper layers, 285 x 95.1 mm, 265 parts, among them Q1 2N7002, SW1 5.2x5.2mm, U1 ATmega32U4-MU, U2 PRTR5V0U2X, Y1 16Mhz

Commit message: 65% variant of voyager60
Parts:
- removed D58, D62: SOD-123, Diodes_SMD:D_SOD-123
- removed G***: LOGO, locallib:ai-ring-6mm
- removed G***: LOGO, locallib:ai-ring-6mm-FancyAss
- removed G***: LOGO, locallib:ai-ring-6mm-FancyAss-Mask
- removed K_ALT2, K_CTRL2, K_RALT3, K_RCTRL3: MX-1.5U, MX_Alps_Hybrid:MX-1.5U-FLIPPED
- removed K_RCTRL2: MX-1.25U, MX_Alps_Hybrid:MX-1.25U
- removed K_RMENU2, K_SPACE5: MX-1.25U, MX_Alps_Hybrid:MX-1.25U-FLIPPED
- removed K_RWIN3, K_SRSHIFT2: MX-1U, MX_Alps_Hybrid:MX-1U
- removed K_SPACE1: MX-7U, MX_Alps_Hybrid:MX-7U-ReversedStabilizers
- removed K_SPACE3: MX-2.25U, MX_Alps_Hybrid:MX-2.25U-ReversedStabilizers
- removed K_SPACE4: MX-2.75U, MX_Alps_Hybrid:MX-2.75U-ReversedStabilizers
- removed K_SRSHIFT1: MX-1.75U, MX_Alps_Hybrid:MX-1.75U
- removed K_WIN2: MX-1U, MX_Alps_Hybrid:MX-1U-FLIPPED
- removed R58, R62: 1k, Resistors_SMD:R_0805
- removed the REF** at (165.1, 69.8)
- added D15: SOD-123, Diodes_SMD:D_SOD-123, B.Cu at (324.6, 108.0)
- added D66: SOD-123, Diodes_SMD:D_SOD-123, B.Cu at (324.6, 31.8)
- added D69: SOD-123, Diodes_SMD:D_SOD-123, B.Cu at (324.8, 50.8)
- added D70: SOD-123, Diodes_SMD:D_SOD-123, B.Cu at (324.6, 69.8)
- added D71: SOD-123, Diodes_SMD:D_SOD-123, B.Cu at (324.6, 89.0)
- added K_DEL1: MX-1U, MX_Alps_Hybrid:MX-1U, F.Cu at (317.5, 31.8)
- added K_DOWN1: MX-1U, MX_Alps_Hybrid:MX-1U, F.Cu at (298.4, 108.0)
- added K_HOM1: MX-1U, MX_Alps_Hybrid:MX-1U, F.Cu at (317.5, 88.9)
- added K_LEFT1: MX-1U, MX_Alps_Hybrid:MX-1U, F.Cu at (279.4, 108.0)
- added K_PGD1: MX-1U, MX_Alps_Hybrid:MX-1U, F.Cu at (317.5, 69.8)
- added K_PGU1: MX-1U, MX_Alps_Hybrid:MX-1U, F.Cu at (317.5, 50.8)
- added K_RIGHT1: MX-1U, MX_Alps_Hybrid:MX-1U, F.Cu at (317.5, 108.0)
- added K_UP1: MX-1U, MX_Alps_Hybrid:MX-1U, F.Cu at (298.4, 88.9)
- added R15: 1k, Resistors_SMD:R_0805, B.Cu at (322.6, 114.0)
- added R66: 1k, Resistors_SMD:R_0805, B.Cu at (322.4, 37.8)
- added R76: 1k, Resistors_SMD:R_0805, B.Cu at (322.4, 57.0)
- added R77: 1k, Resistors_SMD:R_0805, B.Cu at (317.8, 78.3)
- added R78: 1k, Resistors_SMD:R_0805, B.Cu at (321.8, 95.0)
- added REF**: 60_Outline, locallib:65_Outline-Modded, F.Cu at (165.1, 69.8)
- K_RSHIFT1: value MX-2.75U -> MX-1.75U; footprint MX_Alps_Hybrid:MX-2.75U-FLIPPED -> MX_Alps_Hybrid:MX-1.75U
- moved D57 16.9 mm to (305.8, 88.8)
- moved R57 14.1 mm to (302.8, 95.8), turned to 270 degrees
- moved K_RSHIFT1 9.52 mm to (272.3, 88.9)
- moved D30 6.86 mm to (286.2, 108.2)
- moved R30 3.85 mm to (283.2, 113.5)
- moved D65 2.38 mm to (305.6, 108.0)
- renumbered K_RWIN2 to K_RCTRL1
Connections:
- RGB14 pad 2: Net-(RGB14-Pad2) -> (no net)
- U1 pad 1: Net-(U1-Pad1) -> (no net)
- U1 pad 18: Net-(U1-Pad18) -> (no net)
- U1 pad 19: Net-(U1-Pad19) -> COL14
- U1 pad 42: Net-(U1-Pad42) -> (no net)
- U1 pad 8: Net-(U1-Pad8) -> (no net)
- USB1 pad 3: Net-(USB1-Pad3) -> (no net)
- USB1 pad 9: Net-(USB1-Pad9) -> (no net)
Routing:
- net COL14: track 0.00 -> 345.1 mm, vias 0 -> 2
- net LEDGND: track 1409.4 -> 1560.6 mm, vias 11 -> 13
- net ROW0: track 289.8 -> 348.8 mm
- net +5V: track 1795.4 -> 1849.8 mm, vias 13 -> 17
- net ROW1: track 280.9 -> 330.2 mm, vias 2 -> 4
- net ROW3: track 322.7 -> 357.1 mm
- net ROW2: track 359.2 -> 392.9 mm
- net ROW4: track 309.9 -> 330.5 mm
- net COL8: track 365.8 -> 345.9 mm
- net COL4: track 243.6 -> 224.5 mm
- net Net-(K_SPACE2-Pad4): track 29.0 -> 14.6 mm
- net Net-(D61-Pad2): track 29.9 -> 17.0 mm
- net COL6: track 369.3 -> 357.2 mm
- net Net-(D57-Pad2): track 17.8 -> 5.98 mm
- net Net-(D56-Pad2): track 26.8 -> 15.3 mm
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Other:
- board size 285 x 95.1 mm -> 304 x 95.1 mm
